File: Hardware/Aranakin/Aranakin.kicad_sch (KiCad schematic)
At the start: 93 parts, among them J1 Conn_01x03_Socket, J15 5.08-2P-90, J2 Conn_01x03_Socket, J3 Conn_01x03_Socket, J8 Conn_01x03_Socket, K1 G5LE-1, K2 G5LE-1, Q1 2N7002K, Q12 2N7002K, Q2 PMOS, Q3 2N7002K, Q4 2N7002K, Q5 40N02, Q7 2N7002K, U1 XL1509-5.0, U11 HDC1080, U2 AP2112K-3.3, U3 XL1509-12E1, U4 ESP32-C3-Supermini, U5 XL4001, U6 PC817

Commit message: Minor hardware update
Parts:
- added C403: 10u, Capacitor_SMD:C_0805_2012Metric, symbol Device:C
- added PORT1: Conn_01x04_Socket, Connector_Hirose:Hirose_DF13C_CL535-0404-8-51_1x04-1MP_P1.25mm_Vertical, symbol Connector:Conn_01x04_Socket
- renumbered J8 to RELAY1
Connections:
- net +3.3V: now also C403.1, PORT1.1 (Pin_1)
- net GND: now also C403.2, PORT1.4 (Pin_4)
- net Opto: now also U4.23 (GPIO7)
- net SCL: now also PORT1.3 (Pin_3)
- net SDA: now also PORT1.2 (Pin_2)
Other:
- note added: "I2C expansion"
- note added: "Status LED"

Commit message: Added base firmware
Parts:
- removed PWM1: Conn_01x03_Socket, TerminalBlock_Phoenix:TerminalBlock_Phoenix_MKDS-1,5-4_1x04_P5.00mm_Horizontal, symbol Connector:Conn_01x04_Socket
- added F2: Bypass fuse, Fuse:Fuse_1812_4532Metric_Pad1.30x3.40mm_HandSolder, symbol Device:Polyfuse
- added PWM1: 5.08-2P-90, Connector_Phoenix_MSTB:PhoenixContact_MSTBA_2,5_2-G-5,08_1x02_P5.08mm_Horizontal, symbol Connector_Generic:Conn_01x02
- renumbered C11 to C1, C4 to C10, C5 to C11, C8 to C12, C9 to C13, C9 to C14, C10 to C15, C403 to C16, C10 to C17, C12 to C18, C7 to C2, C55 to C3, C1 to C4, C6 to C5, C2 to C6, C3 to C7, C100 to C8, C28 to C9, D27 to D1, D9 to D10, D10 to D11, D11 to D12, D8 to D13, D2 to D14, D4 to D2, D26 to D3, D6 to D4, D1 to D5, D3 to D6, D5 to D7, D7 to D8, D7 to D9, J15 to J1, L6 to L1, L1 to L2, L1 to L3, L3 to L4, Q12 to Q1, Q1 to Q3, Q7 to Q4, Q3 to Q5, Q4 to Q6, Q5 to Q7, R84 to R1, R6 to R10, R8 to R12, R10 to R13, R70 to R14, R68 to R15, R18 to R17, R9 to R18, R85 to R2, R17 to R21, R5 to R22, R15 to R23, R12 to R24, R13 to R25, R14 to R26, R83 to R3, R36 to R5, R1 to R6, R2 to R7, R3 to R8, R7 to R9, RELAY1 to RL1, J1 to RL2, U5 to U1, U1 to U2, U2 to U3, U11 to U4, U4 to U5, U3 to U6, U6 to U7
Connections:
- net +5V: now also U5.16 (5V); no longer U5.13 (5V), U5.14 (5V)
- net 12V_enable: now also U5.11 (GPIO2); no longer U5.4 (GPIO2)
- net ADC0: now also U5.13 (GPIO4); no longer U5.9 (GPIO0)
- net CC_CH0: now also U5.1 (GPIO5); no longer U5.21 (GPIO5)
- net GND: no longer U5.1 (GND), U5.12 (GND), U5.16 (GND), U5.19 (GND), U5.24 (GND), U5.27 (GND), U5.30 (GND), U5.6 (GND), U5.8 (GND)
- net LED_PIN: now also U5.12 (GPIO3); no longer U5.10 (GPIO1)
- net Opto: now also U5.6 (GPIO10); no longer U5.23 (GPIO7)
- net RELAY0_PIN: now also U5.9 (GPIO0); no longer U5.20 (GPIO4)
- net RELAY1_PIN: now also U5.10 (GPIO1); no longer U5.5 (GPIO3)
- net SCL: now also U5.4 (GPIO8); no longer U5.26 (GPIO9)
- net SDA: now also U5.3 (GPIO7); no longer U5.25 (GPIO8)
- net VCC: now also F2.1; no longer D13.1 (K)
- net Vin: now also D13.1 (K), PWM1.2 (Pin_2)
- net openDrain: now also U5.2 (GPIO6); no longer U5.22 (GPIO6)
- net relayPWR: now also F2.2
- net at D13.2 (A), Q7.3 (D): now also PWM1.1 (Pin_1)
- removed net 3V3: JP1.2 (B), U5.2 (3V3), U5.3 (3V3)
- new net: JP1.2 (B), U5.14 (3V3)

Commit message: Hardware update
Parts:
- removed C11: 10u, Capacitor_SMD:C_0805_2012Metric, symbol Device:C
- removed C12: 100nF, Capacitor_SMD:C_0805_2012Metric, symbol Device:C
- removed C14, C17: 100uF, Capacitor_SMD:C_Elec_6.3x7.7, symbol Device:C_Polarized
- removed L3: 22n, Inductor_SMD:L_0805_2012Metric, symbol Device:L
- removed R3, R8: 2k, Resistor_SMD:R_0402_1005Metric_Pad0.72x0.64mm_HandSolder, symbol 1_Library_GF:R_SMD_0805
- added J4: 1Wire, TerminalBlock:TerminalBlock_Xinya_XY308-2.54-3P_1x03_P2.54mm_Horizontal, symbol Connector:Conn_01x03_Socket
- added JP2: SolderJumper_3_Open, Jumper:SolderJumper-3_P1.3mm_Open_RoundedPad1.0x1.5mm, symbol Jumper:SolderJumper_3_Open
- added R27: 10k, Resistor_SMD:R_0805_2012Metric, symbol Device:R
- added R3, R8: 2.2k, Resistor_SMD:R_0805_2012Metric, symbol Device:R
- C1, C3, C4, C5, CC1, D4, J2, L1, Q4, R10, R12, R14, R15, R9, RTC1, U1: now not fitted; now left out of the parts list
- C9: value 100n -> 100nF; footprint Capacitor_SMD:C_0402_1005Metric -> Capacitor_SMD:C_0805_2012Metric; LCSC C1525 -> C49678; Manufacturer  (none) -> YAGEO; Mfr. Part Number (none) -> CC0805KRX7R9BB104; Observations (none) -> Accepts other suppliers
- R21: value 1k -> 10k; LCSC C95781 -> C17414
- U7: value PC817 -> PC817XI; footprint Package_DIP:SMDIP-4_W7.62mm -> Package_DIP:DIP-4_W8.89mm_SMDSocket_LongPads; LCSC C5451664 -> (none); Manufacturer  (none) -> Slkor; Mfr. Part Number (none) -> PC817B; Observations (none) -> Accepts other suppliers
Connections:
- net +3.3V: now also C9.2, J4.1 (Pin_1), R27.2; no longer C9.1
- net CC_CH0: no longer U5.1 (GPIO5)
- net GND: now also C9.1, J4.3 (Pin_3); no longer C9.2
- net LED_PIN: now also U5.6 (GPIO10); no longer U5.12 (GPIO3)
- net Opto: now also U5.12 (GPIO3); no longer U5.6 (GPIO10)
- net Vin: now also JP2.3 (B); no longer D13.1 (K), PWM1.2 (Pin_2)
- net relayPWR: now also R21.2, JP2.1 (A); no longer R21.1
- net at D8.2 (A): now also R21.1; no longer R21.2
- net at D5.2 (A), K2.2, Q3.3 (D): now also R8.1
- net at D6.1 (K): now also R8.2
- net at D1.2 (A), K1.2, Q1.3 (D): now also R3.1
- net at D3.1 (K): now also R3.2
- net ADC0 renamed ADC
- new net: D13.1 (K), JP2.2 (C), PWM1.2 (Pin_2)
- new net 1Wire: J4.2 (Pin_2), R27.1, U5.1 (GPIO5)
Other:
- note added: "1Wire"
- moved on the sheet: D12, D13, PWM1, Q6, Q7, R24, R25

Commit message: Added first layout and fabrication files
Parts:
- added PORT2: Conn_01x03_Socket, Connector_PinHeader_2.54mm:PinHeader_1x03_P2.54mm_Vertical, symbol Connector:Conn_01x03_Socket
Connections:
- net GND: now also PORT2.3 (Pin_3)
- net at U5.7 (GPIO20/U0RXD): now also PORT2.1 (Pin_1)
- net at U5.8 (GPIO21/U0TXD): now also PORT2.2 (Pin_2)
Changed lines of the file:
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@@
 	(wire
 		(pts
+			(xy 195.58 109.22) (xy 205.74 109.22)
+		)
+		(stroke
+			(width 0)
+			(type default)
+		)
+	)
+	(wire
+		(pts
 			(xy 49.53 110.49) (xy 50.8 110.49)
 		)
@@
 	(wire
 		(pts
+			(xy 204.47 113.03) (xy 204.47 111.76)
+		)
+		(stroke
+			(width 0)
+			(type default)
+		)
+	)
+	(wire
+		(pts
 			(xy 172.72 33.02) (xy 176.53 33.02)
 		)
@@
 	(wire
 		(pts
+			(xy 204.47 111.76) (xy 205.74 111.76)
+		)
+		(stroke
+			(width 0)
+			(type default)
+		)
+	)
+	(wire
+		(pts
 			(xy 29.21 124.46) (xy 33.02 124.46)
 		)
@@
 	(wire
 		(pts
+			(xy 195.58 106.68) (xy 205.74 106.68)
+		)
+		(stroke
+			(width 0)
+			(type default)
+		)
+	)
+	(wire
+		(pts
 			(xy 261.62 153.67) (xy 264.16 153.67)
 		)
@@
 		(on_board yes)
 		(dnp no)
-		(fields_autoplaced yes)
 		(property "Reference" "#PWR054"
 			(at 200.66 116.84 0)
@@
 		)
 		(property "Value" "+3.3V"
-			(at 200.66 107.95 0)
+			(at 196.342 111.506 0)
 			(effects
 				(font
@@
 	)
 	(symbol
+		(lib_id "power:GND")
+		(at 204.47 113.03 0)
+		(unit 1)
+		(exclude_from_sim no)
+		(in_bom yes)
+		(on_board yes)
+		(dnp no)
+		(fields_autoplaced yes)
+		(property "Reference" "#PWR040"
+			(at 204.47 119.38 0)
+			(effects
+				(font
+					(size 1.27 1.27)
+				)
+				(hide yes)
+			)
+		)
+		(property "Value" "GND"
+			(at 204.47 118.11 0)
+			(effects
+				(font
+					(size 1.27 1.27)
+				)
+			)
+		)
+		(property "Footprint" ""
+			(at 204.47 113.03 0)
+			(effects
+				(font
+					(size 1.27 1.27)
+				)
+				(hide yes)
+			)
+		)
+		(property "Datasheet" ""
+			(at 204.47 113.03 0)
+			(effects
+				(font
+					(size 1.27 1.27)
+				)
+				(hide yes)
+			)
+		)
+		(property "Description" "Power symbol creates a global label with name \"GND\" , ground"
+			(at 204.47 113.03 0)
+			(effects
+				(font
+					(size 1.27 1.27)
+				)
+				(hide yes)
+			)
+		)
+		(pin "1"
+		)
+		(instances
+			(project "Aranakin"
+				(path "/435bb94e-d379-4041-9433-e08282ea3ba2"
+					(reference "#PWR040")
+					(unit 1)
+				)
+			)
+		)
+	)
+	(symbol
 		(lib_id "Device:R")
 		(at 132.08 87.63 0)
@@
 					(unit 1)
 				)
+			)
+		)
+	)
+	(symbol
+		(lib_id "Connector:Conn_01x03_Socket")
+		(at 210.82 109.22 0)
+		(unit 1)
+		(exclude_from_sim no)
+		(in_bom yes)
+		(on_board yes)
+		(dnp no)
+		(property "Reference" "PORT2"
+			(at 205.74 103.632 0)
+			(effects
+				(font
+					(size 1.27 1.27)
+				)
+				(justify left)
+			)
+		)
+		(property "Value" "Conn_01x03_Socket"
+			(at 212.09 110.4899 0)
+			(effects
+				(font
+					(size 1.27 1.27)
+				)
+				(justify left)
+				(hide yes)
+			)
+		)
+		(property "Footprint" "Connector_PinHeader_2.54mm:PinHeader_1x03_P2.54mm_Vertical"
+			(at 210.82 109.22 0)
+			(effects
+				(font
+					(size 1.27 1.27)
+				)
+				(hide yes)
+			)
+		)
+		(property "Datasheet" "~"
+			(at 210.82 109.22 0)
+			(effects
+				(font
+					(size 1.27 1.27)
+				)
+				(hide yes)
+			)
+		)
+		(property "Description" "Generic connector, single row, 01x03, script generated"
+			(at 210.82 109.22 0)
+			(effects
+				(font
+					(size 1.27 1.27)
+				)
+				(hide yes)
+			)
+		)
+		(pin "2"
+		)
+		(pin "3"
+		)
+		(pin "1"
+		)
+		(instances
+			(project "Aranakin"
+				(path "/435bb94e-d379-4041-9433-e08282ea3ba2"
+					(reference "PORT2")
+					(unit 1)
+				)
