File: Hardware/Echoes_of_Termina/Echoes_of_Termina.kicad_sch (KiCad schematic)
At the start: 72 parts, among them J1 Conn_01x03_Socket, J2 USB_C_Receptacle_USB2.0_8P, J3 Conn_01x02_Socket, J4 Conn_01x02_Socket, Q1 PMOS, Q2 2N7002K, U1 AP2112K-3.3, U1 TP4056, U2 MAX98357A, U3 ESP32-WROOM-32, U4 MAX98357A

Commit message: First PCB sketch for Echoes of Termina
Parts:
- removed C4: 220uF, Capacitor_SMD:CP_Elec_6.3x7.7, symbol Device:C_Polarized
- added C11: 220uF, Capacitor_SMD:CP_Elec_8x10.5, symbol Device:C_Polarized
- added D9: SS14, Diode_SMD:D_SMA, symbol Diode:SS14
- added H1, H2, H3, H4: MountingHole, MountingHole:MountingHole_3.2mm_M3, symbol Mechanical:MountingHole
- added Q3: PMOS, Package_TO_SOT_SMD:SOT-23_Handsoldering, symbol Simulation_SPICE:PMOS
- added R25: 100k, Resistor_SMD:R_0805_2012Metric, symbol Device:R
- added R26, R27: 2.2k, Resistor_SMD:R_0805_2012Metric, symbol Device:R
- BT3: renamed from BT1; LCSC C455246 -> C2888502
- BT4: LCSC C455246 -> C2888502
- C1: renamed from C3; LCSC C15850 -> C162422
- C12: renamed from C26; value 100nF -> 100n
- C14: renamed from C48; value 100nF -> 100n
- C16: renamed from C6; value 100nF -> 100n
- C17: renamed from C10; LCSC C15850 -> C162422
- C2: LCSC C2909631 -> C49678
- C3: renamed from C1; LCSC C2909631 -> C49678
- C6: renamed from C38; footprint Capacitor_SMD:C_0402_1005Metric_Pad0.74x0.62mm_HandSolder -> Capacitor_SMD:C_0805_2012Metric; LCSC C85858 -> C49678
- C7: renamed from C34; Link (none) -> https://www.lcsc.com/product-detail/C2162971.html?; Observations 35V 800mA 6.3x7.7mm -> 35V 850mA 8x10.5mm
- C8: renamed from C18; value 100nF -> 100n
- C9: renamed from C39; footprint Capacitor_SMD:C_0402_1005Metric_Pad0.74x0.62mm_HandSolder -> Capacitor_SMD:C_0805_2012Metric; LCSC C85858 -> C49678
- D8: renamed from D3; LCSC C2909920 -> C2480
- PORT1: renamed from PORT2; footprint Library:Hirose_DF13C_CL535-0404-8-51_1x04-1MP_P1.25mm_Vertical -> Connector_Hirose:Hirose_DF13C_CL535-0404-8-51_1x04-1MP_P1.25mm_Vertical
- R12: renamed from R50; footprint Resistor_SMD:R_0402_1005Metric_Pad0.72x0.64mm_HandSolder -> Resistor_SMD:R_0805_2012Metric; LCSC C25744 -> C17414
- R13: renamed from R51; footprint Resistor_SMD:R_0402_1005Metric_Pad0.72x0.64mm_HandSolder -> Resistor_SMD:R_0805_2012Metric; LCSC C25744 -> C17414
- R14: renamed from R52; footprint Resistor_SMD:R_0402_1005Metric_Pad0.72x0.64mm_HandSolder -> Resistor_SMD:R_0805_2012Metric; LCSC C25744 -> C17414
- R15: renamed from R53; footprint Resistor_SMD:R_0402_1005Metric_Pad0.72x0.64mm_HandSolder -> Resistor_SMD:R_0805_2012Metric; LCSC C25744 -> C17414
- TF1: footprint Library:TF-SMD_TF-CARD-XG8P-H1.5 -> Aleoexpress:TF-SMD_TF-CARD-XG8P-H1.5
- renumbered C40 to C10, C43 to C13, C5 to C15, C36 to C4, C37 to C5, D30 to D2, D31 to D3, D2 to D4, D4 to D5, D32 to D6, D33 to D7, J2 to J1, J1 to J2, JP3 to JP1, JP1 to JP2, L2 to L1, PORT1 to PORT2, R2 to R1, R6 to R11, R11 to R16, R16 to R17, R12 to R18, R13 to R19, R3 to R2, R14 to R20, R2 to R21, R15 to R22, R25 to R23, R7 to R24, R1 to R3, R73 to R6, R74 to R7, U1 to U2, U2 to U5
Connections:
- net Boot is gone; now on net PROG: BT4.2
- net +3.3V: now also R26.2, R27.2
- net +5V: now also D9.2 (A), Q3.1 (G), R25.2
- net GND: now also C11.2, R25.1
- net I2S_BCLK: now also U3.28 (IO17); no longer U3.30 (IO18)
- net I2S_LRC: now also U3.30 (IO18); no longer U3.28 (IO17)
- net SCL: now also R27.1
- net SDA: now also R26.1
- net V_REG: now also C11.1, Q3.3 (D); no longer C13.1, C14.2, C15.1, C16.2, JP1.3 (B), JP2.3 (B), R23.1, R24.1, U4.7 (Out+), U5.7 (Out+)
- net at J3.1 (Pin_1): now also U4.9 (Out-); no longer U4.7 (Out+)
- net at J4.1 (Pin_1): now also U5.9 (Out-); no longer U5.7 (Out+)
- new net V_SPK: C13.1, C14.2, C15.1, C16.2, D9.1 (K), JP1.3 (B), JP2.3 (B), Q3.2 (S), R23.1, R24.1, U4.7 (VIN), U5.7 (VIN)
Other:
- note added: "Cutoff Q2 pulls Vg(Q3) high PMOS blocks battery discharge Button trigger activates Q2 Q3 saturates, V_REG = V_BAT - 200mV ESP32 boots, drive GPIO25 high to latch power on"
- note removed: "Cutoff Q2 pulls Q3 up PMOS blocks battery discharge Button trigger activates Q2 Q3 saturates, V_REG = V_BAT - 200mV Supermini boots, drive GPIO4 high to latch power on"
- moved on the sheet: BT4, D5, R11, TOUCH1

Commit message: Echoes layout for revision before fabrication
Parts:
- D1: now not fitted; now left out of the parts list
- H3, H4: now not fitted
Connections:
- net Button_GPIO: now also U3.26 (IO4); no longer U3.11 (IO26)
- net Strip_out: now also U3.10 (IO25); no longer U3.16 (IO13)
- net V_SPK: now also C7.1
- net latch_enable: now also U3.16 (IO13); no longer U3.10 (IO25)
- net at D1.1 (K), D4.1 (K), U2.1 (VIN)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: no longer C7.1
Other:
- note added: "Cutoff Q2 pulls Vg(Q1) high PMOS blocks battery discharge Button trigger activates Q2 Q1 saturates, V_REG = V_BAT - 200mV ESP32 boots, drive GPIO25 high to latch power on"
- note removed: "Cutoff Q2 pulls Vg(Q3) high PMOS blocks battery discharge Button trigger activates Q2 Q3 saturates, V_REG = V_BAT - 200mV ESP32 boots, drive GPIO25 high to latch power on"
- moved on the sheet: C13, C14, C15, C16, C7, H1, H2, J3, J4, JP1, JP2, R23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
