File: Hardware/GNSS_ZED/GNSS_ZED.kicad_sch (KiCad schematic)
At the start: 78 parts, among them J1 5.08-2P-90, J2 USB_C_Receptacle_USB2.0_8P, J3 Conn_02x12_Odd_Even, J4 Conn_02x12_Odd_Even, J6 5.08-2P-90, Q1 PMOS, Q18 PMOS, U1 ESP32-S3-WROOM-1, U2 AP2112K-3.3, U2 XL1509-5.0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

Commit message: GNSS_ZED update
Parts:
- removed D43: SS14, Diode_SMD:D_SMA, symbol Diode:SS14
- removed Q18: PMOS, Package_TO_SOT_SMD:SOT-223-3_TabPin2, symbol Simulation_SPICE:PMOS
- removed R112, R17, R18, R19: 100k, Resistor_SMD:R_0805_2012Metric, symbol Device:R
- removed R33: 8.2k, Resistor_SMD:R_0805_2012Metric, symbol Device:R
- added C7: 10u, Capacitor_SMD:C_0805_2012Metric, symbol Device:C
- added D5: SS14, Diode_SMD:D_SMA, symbol Diode:SS14
- added GNSS1, PORT2: Conn_01x04_Socket, Connector_Hirose:Hirose_DF13C_CL535-0404-8-51_1x04-1MP_P1.25mm_Vertical, symbol Connector:Conn_01x04_Socket
- added Q2: PMOS, Package_TO_SOT_SMD:SOT-23_Handsoldering, symbol Simulation_SPICE:PMOS
- added R11: 100k, Resistor_SMD:R_0805_2012Metric, symbol Device:R
- added R12, R13, R14: 10k, Resistor_SMD:R_0805_2012Metric_Pad1.20x1.40mm_HandSolder, symbol Device:R
- R24: value 8.2k -> 9.1k
Connections:
- net ADC1_0 is gone; now on net ADC: C8.2
- net +5V: now also C2.1, D2.1 (VDD), C7.1, GNSS1.1 (Pin_1), PORT2.1 (Pin_1)
- net ADC: now also U1.19 (IO11), R13.2, R14.1
- net GND: now also C7.2, GNSS1.4 (Pin_4), PORT2.4 (Pin_4), R11.2, R14.2
- net PCH0: now also Q2.3 (D), R12.1
- net Status_LED: now also U1.24 (IO47)
- net TFT_BCK: now also J3.17 (Pin_17), J4.17 (Pin_17)
- net TFT_CS: now also J3.11 (Pin_11), J4.11 (Pin_11)
- net TFT_DC: now also J3.13 (Pin_13), J4.13 (Pin_13)
- net TFT_MISO: now also J3.21 (Pin_21), J4.21 (Pin_21)
- net TFT_MOSI: now also J3.19 (Pin_19), J4.19 (Pin_19)
- net TFT_RST: now also J3.15 (Pin_15), J4.15 (Pin_15)
- net TFT_SCK: now also J3.23 (Pin_23), J4.23 (Pin_23)
- net TOUCH_CS: now also J3.7 (Pin_7), J4.7 (Pin_7)
- net TOUCH_INT: now also J3.9 (Pin_9), J4.9 (Pin_9)
- net VCC: now also D5.2 (A), Q2.1 (G), R11.1
- net V_REG: now also U2.1 (VIN), D5.1 (K), Q2.2 (S); no longer C2.1, D2.1 (VDD)
- net at JP1.1 (A): now also R12.2
- net SDA1: now reaches U1.21 (IO13)
- net SDA1: now also GNSS1.2 (Pin_2)
- net SCL1: now reaches U1.22 (IO14)
- net SCL1: now also GNSS1.3 (Pin_3)
- net RX0: now reaches U1.36 (RXD0)
- net RX0: now also PORT1.3 (Pin_3)
- net TX0: now reaches U1.37 (TXD0)
- net TX0: now also PORT1.2 (Pin_2)
- net at R16.1: now also R13.1
- net SCL renamed SCL2
- net SCL2: now also PORT2.3 (Pin_3); no longer PORT1.3 (Pin_3)
- net SDA renamed SDA2
- net SDA2: now also PORT2.2 (Pin_2); no longer PORT1.2 (Pin_2)
Other:
- note added: "ADC_ATTEN_DB_2_5 V(ADC)<1250mV V_reg(max) = 13V V(ADC)/V_reg <= 0.1"
- note added: "GPTO"
- note added: "In case of external supply present, PMOS blocks battery drain"
- note added: "Serial expansion"
- note added: "VOUT=1.235*(1+RB/RA) 12.5V: RB/RA = 9.1 7.3V: RB/RA = 4.9 10k//9.1k = 4.7k"
- note removed: "ADC_ATTEN_DB_2_5 V(ADC)<1050mV V_reg(max) = 4.2V V(ADC)/V_reg <= 0.25"
- note removed: "PMOS blocks battery drain in case of 5V present"
- note removed: "VOUT=1.235*(1+RB/RA) 7 < VOUT < 13 5 < RB/RA < 10"
- moved on the sheet: C8, D16, J3, J4, R16, R32
